File: DC Load.kicad_sch (KiCad schematic)
At the start: 27 parts, among them IC1 AD711JRZ-REEL, IC2 AD633JRZ, IC3 ISO124P, IC5 L78L08ABZTR, Q1 KSC2383YTA, Q2 STW12N120K5, U1 TMCS1133C9AQDVGR

Commit message: Started putting together the full circuit
Parts:
- removed A1: Arduino_Nano_v3.x, Module:Arduino_Nano, symbol MCU_Module:Arduino_Nano_v3.x
- removed C1, C2, C6, C7: 1u, symbol Device:C
- removed C12, C13, C3, C4, C5, C8, C9, C? (x2): 0.1u, symbol Device:C
- removed IC1: AD711JRZ-REEL, SOIC127P600X175-8N, symbol AD711JRZ-REEL:AD711JRZ-REEL
- removed IC2: AD633JRZ, SOIC127P600X175-8N, symbol AD633JRZ:AD633JRZ
- removed IC3: ISO124P, DIP794W56P254L2000H533Q16N, symbol ISO124P:ISO124P
- removed IC5: L78L08ABZTR, L78L08ABZTR, symbol L78L08ABZTR:L78L08ABZTR
- removed IC?: L78L05ACZ, L78L05ACZ, symbol L78L05ACZ:L78L05ACZ
- removed Q1: KSC2383YTA, TO-92-3, symbol KSC2383YTA:KSC2383YTA
- removed Q2: STW12N120K5, TO545P515X1560X2445-3P, symbol STW12N120K5:STW12N120K5
- removed R1: 10k, symbol Device:R
- removed R4: 10M, symbol Device:R
- removed R5: 160k, symbol Device:R
- removed U1: TMCS1133C9AQDVGR, TMCS1133C9AQDVGR:DVG0010A_PMCS1133A1AQDVGR_TEX, symbol TMCS1133C9AQDVGR:TMCS1133C9AQDVGR
- added A1: Arduino_Nano_ESP32, Module:Arduino_Nano, symbol MCU_Module:Arduino_Nano_ESP32
- added D1: IXBOD1-08, IXBOD108, symbol IXBOD1-08:IXBOD1-08
- added IC1, IC2, IC6: REF7050QDGKR, SOP65P490X110-8N, symbol REF7050QDGKR:REF7050QDGKR
- added IC3: MAX5719GSD+, SOIC127P600X175-14N, symbol MAX5719GSD+:MAX5719GSD+
- added IC4: AD7175-2BRUZ, SOP65P640X120-24N, symbol AD7175-2BRUZ:AD7175-2BRUZ
- added IC5, IC8: OPA210IDGKR, SOP65P490X110-8N, symbol OPA210IDGKR:OPA210IDGKR
- added IC7: INA826AID, SOIC127P600X175-8N, symbol INA826AID:INA826AID
- added IC9: INA296A3IDDFR, SOT65P280X110-8N, symbol INA296A3IDDFR:INA296A3IDDFR
- added Q1: MSC017SMA120B4N, Package_TO_SOT_THT:TO-247-4_Vertical, symbol MSC017SMA120:MSC017SMA120B4N
- added R1: PCS-0R0047D1, symbol Device:R_Shunt_US
- added RV1: Current_Sense_Amp_Ref_Adjust, symbol Device:R_Potentiometer_Trim
- R2: value 10k -> 2M
- R3: value 460 -> 15.8k
Connections:
- net +5V: now also IC3.14 (VDD), IC4.7 (AVDD1), IC9.6 (VS)
- net GND: now also IC1.3 (GND_1), IC1.4 (GND_2), IC1.5 (GND_3), IC1.8 (GND_4), IC2.3 (GND_1), IC2.4 (GND_2), IC2.5 (GND_3), IC2.8 (GND_4), IC3.12 (DGND), IC3.3 (AGNDF), IC3.4 (AGNDS), IC4.17 (DGND), IC4.2 (REF-), IC4.6 (AVSS), IC5.4 (V-), IC6.3 (GND_1), IC6.4 (GND_2), IC6.5 (GND_3), IC6.8 (GND_4), IC7.5 (-VS), IC8.4 (V-), IC9.2 (GND), Q1.3 (DS), RV1.1; no longer R3.2
- net in+: now reaches R2.1
- net in+: now also D1.2 (K), Q1.1 (D)
- net Voltage Sense +: now reaches R3.1
- net Voltage Sense +: now also R2.2, IC7.4 (+IN)
- new net: A1.29 (GND), A1.4 (GND)
- new net: Q1.2 (S), R1.1
- new net: IC3.2 (OUT), IC5.3 (+IN)
- new net: IC1.6 (OUTS), IC3.5 (REFS)
- new net: IC1.7 (OUTF), IC3.6 (REFF)
- new net: IC2.6 (OUTS), IC2.7 (OUTF), IC4.3 (REF+)
- new net: IC8.3 (+IN), RV1.2
- new net: IC6.6 (OUTS), IC6.7 (OUTF), RV1.3
- new net +21V: IC5.7 (V+)
- new net +3.3V: IC4.16 (IOVDD), IC4.8 (AVDD2)
- new net +3.3v: IC7.8 (+VS), IC8.7 (V+)
- new net +5.5V: IC1.1 (EN), IC1.2 (VIN), IC2.1 (EN), IC2.2 (VIN), IC6.1 (EN), IC6.2 (VIN)
- new net Current Sense +: IC9.8 (IN+), R1.2
- new net Current Sense -: IC9.1 (IN-), R1.3
- new net Current Sense Amp Out: IC4.24 (AIN3), IC9.5 (OUT)
- new net Current Sense Amp Ref: IC8.6 (OUT), IC9.3 (REF2), IC9.7 (REF1)
- new net Gate Drive +: IC5.6 (OUT), Q1.4 (G)
- new net Gate Drive CS: IC3.7 (~{CS})
- new net Gate Drive Din: IC3.10 (DIN)
- new net Gate Drive LDAC: IC3.11 (~{LDAC})
- new net Gate Drive SCLK: IC3.8 (SCLK)
- new net Sense Amp Ref: IC4.21 (AIN0), IC4.23 (AIN2), IC7.6 (REF), IC8.2 (-IN)
- new net Sense CS: IC4.14 (~{CS})
- new net Sense Din: IC4.12 (DIN)
- new net Sense Dout: IC4.11 (DOUT/~{RDY})
- new net Sense SCLK: IC4.13 (SCLK)
- new net Voltage Sense -: D1.1 (A), IC7.1 (-IN), R1.4, R3.2
- new net Voltage Sense Amp Out: IC4.22 (AIN1), IC7.7 (VOUT)
- no-connect marks 31 -> 14
Other:
- note added: "Gate Drive"
- note added: "Load"
- note added: "Sense"

Commit message: Updated the schematic for the control loop
Parts:
- added C1, C16, C17, C35, C36, C45, C57: 1u, symbol Device:C
- added C10, C23, C29, C37, C38, C48, C49, C51, C52, C53, C55, C56, C8, C9: 0.1u, symbol Device:C
- added C11, C15, C18, C19, C20, C21, C22, C28, C32, C39, C40, C47, C7: .1u, symbol Device:C
- added C12, C14, C26, C30, C46, C50, C54, C6: 10u, symbol Device:C
- added C13, C27: 180p, symbol Device:C
- added C2, C4: 0.47u, symbol Device:C
- added C24: 1n, symbol Device:C
- added C25: 0.01u, symbol Device:C
- added C3, C5: 0.33u, symbol Device:C
- added C31: 540p, symbol Device:C
- added C33, C34: 680p, symbol Device:C
- added C41, C42, C43, C44: 270p, symbol Device:C
- added D1: HPZR-C21-QX, HPZRC21QX, symbol HPZR-C21-QX:HPZR-C21-QX
- added IC12: ISO7740FQDBQRQ1, SOP64P600X175-16N, symbol ISO7740FQDBQRQ1:ISO7740FQDBQRQ1
- added IC13, IC9: ISO7741FQDBQRQ1, SOP64P600X175-16N, symbol ISO7741FQDBQRQ1:ISO7741FQDBQRQ1
- added IC2: L78L06ACD13TR, SOIC127P600X175-8N, symbol L78L06ACD13TR:L78L06ACD13TR
- added IC3: L78L05ACD13TR, SOIC127P600X175-8N, symbol L78L05ACD13TR:L78L05ACD13TR
- added IC4, IC5: L78L33ACD13TR, SOIC127P600X175-8N, symbol L78L33ACD13TR:L78L33ACD13TR
- added L1: 47u, symbol Device:L
- added L2: 68u, symbol Device:L
- added PS1: NKE1212DC, NKE0503DC, symbol NKE1212DC:NKE1212DC
- added PS2: NMG1224SC, NMG0524SC, symbol NMG1224SC:NMG1224SC
- added PS3, PS4: TBA_1-1219, TBA1, symbol TBA_1-1219:TBA_1-1219
- added R1, R2: 9.09k, symbol Device:R
- added RV1: Gate_Drive_Amp_Gain_Adjust 4.7k, symbol Device:R_Potentiometer_Trim
- IC14: renamed from IC7; EVBoard (none) -> https://www.ti.com/lit/ug/sbou115c/sbou115c.pdf?ts=17380260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
- renumbered D1 to D2, IC5 to IC10, IC6 to IC11, IC8 to IC15, IC9 to IC16, IC3 to IC6, IC2 to IC7, IC4 to IC8, R1 to R3, R2 to R4, R3 to R5, RV1 to RV2
Connections:
- net Current Sense Amp Ref is gone; now on net Sense Amp Ref: IC15.6 (OUT), IC16.3 (REF2), IC16.7 (REF1)
- net +3.3V: now also C29.1, C48.1, C53.1, IC12.1 (VCC1), IC13.10 (EN2), IC13.16 (VCC2), IC5.1 (VOUT), IC9.1 (VCC1), IC9.7 (EN1); no longer IC8.16 (IOVDD), IC8.8 (AVDD2)
- net Current Sense Amp Out: now also C33.2, C41.1
- net GND: now also A1.29 (GND), A1.4 (GND), C29.2, C48.2, C53.2, IC12.2 (GND1_1), IC12.8 (GND1_2), IC13.15 (GND2_2), IC13.9 (GND2_1), IC5.2 (GND_1), IC5.3 (GND_2), IC5.6 (GND_3), IC5.7 (GND_4), IC9.2 (GND1_1), IC9.8 (GND1_2), PS1.1 (-VIN), PS2.2 (-VIN), PS3.1 (-VIN_(GND)), PS4.1 (-VIN_(GND)); no longer IC1.3 (GND_1), IC1.4 (GND_2), IC1.5 (GND_3), IC1.8 (GND_4), IC10.4 (V-), IC11.3 (GND_1), IC11.4 (GND_2), IC11.5 (GND_3), IC11.8 (GND_4), IC14.5 (-VS), IC15.4 (V-), IC16.2 (GND), IC6.12 (DGND), IC6.3 (AGNDF), IC6.4 (AGNDS), IC7.3 (GND_1), IC7.4 (GND_2), IC7.5 (GND_3), IC7.8 (GND_4), IC8.17 (DGND), IC8.2 (REF-), IC8.6 (AVSS), Q1.3 (DS), RV2.1
- net Gate Drive +: now also C31.2, D1.1 (K), R1.2
- net Gate Drive Din: now also IC12.12 (OUTC)
- net Gate Drive SCLK: now also IC12.13 (OUTB)
- net Sense Amp Ref: now also C33.1, C34.1, C42.1, C44.1
- net Sense Din: now also IC9.12 (OUTC)
- net Sense SCLK: now also IC9.13 (OUTB)
- net Voltage Sense Amp Out: now also C34.2, C43.1
- net Sense ~{Error} uC: now reaches A1.10 (D7)
- net Sense ~{Error} uC: now also IC13.14 (OUTA)
- net Gate Drive ~{LDAC} uC: now reaches A1.11 (D8)
- net Gate Drive ~{LDAC} uC: now also IC12.6 (IND)
- net Gate Drive ~{CS} uC: now reaches A1.12 (D9)
- net Gate Drive ~{CS} uC: now also IC12.3 (INA)
- net Sense ~{CS} uC: now reaches A1.13 (D10/CS)
- net Sense ~{CS} uC: now also IC9.3 (INA)
- net COPI uC: now reaches A1.14 (D11/COPI)
- net COPI uC: now also IC12.5 (INC), IC9.5 (INC)
- net CIPO uC: now reaches A1.15 (D12/CIPO)
- net CIPO uC: now also IC9.6 (OUTD)
- net SCLK uC: now reaches A1.16 (D13/SCK)
- net SCLK uC: now also IC12.4 (INB), IC9.4 (INB)
- net +12V: now reaches A1.30 (VIN)
- net +12V: now also IC5.8 (VIN), PS1.4 (+VIN), PS2.1 (+VIN), PS3.2 (+VIN_(VCC)), PS4.2 (+VIN_(VCC))
- net Gate Drive DAC Out: now reaches IC10.3 (+IN), IC6.2 (OUT)
- net Gate Drive DAC REFS: now reaches IC1.6 (OUTS), IC6.5 (REFS)
- net Gate Drive DAC REFF: now reaches IC1.7 (OUTF), IC6.6 (REFF)
- net Gate Drive DAC REFF: now also C11.2, C12.2, C13.1
- net ADC Ref+: now reaches IC7.6 (OUTS), IC7.7 (OUTF), IC8.3 (REF+)
- net ADC Ref+: now also C22.1, C26.2, C28.2
- net at IC15.3 (+IN): now also RV2.3, R2.1; no longer RV2.2
- net at IC11.6 (OUTS), IC11.7 (OUTF): now also C46.2, C47.2, R2.2; no longer RV2.3
- net at IC10.2 (-IN): now also C31.1, R1.1, RV1.3
- net Sense ~{Error}: now reaches IC8.15 (~{SYNC}/~{ERROR})
- net Sense ~{Error}: now also IC13.3 (INA)
- net at IC8.18 (REGCAPD): now also C35.2, C39.2
- net Sense GPIO1: now reaches IC8.19 (GPIO0)
- net Sense GPIO0: now reaches IC8.20 (GPIO1)
- net at IC8.5 (REGCAPA): now also C16.2, C18.2
- net +21V renamed +21V Isolated
- net +21V Isolated: now also C1.2, C38.2, C45.2, L1.1
- net +3.3v renamed +3.3V Isolated
- net +3.3V Isolated: now also IC8.16 (IOVDD), IC8.8 (AVDD2), C21.1, C36.1, C37.1, C40.1, C49.1, C52.1, C55.2, C57.2, C8.2, IC12.10 (EN2), IC12.16 (VCC2), IC13.1 (VCC1), IC4.1 (VOUT), IC9.10 (EN2), IC9.16 (VCC2); no longer IC14.8 (+VS)
- net +5.5V renamed +6V Isolated
- net +6V Isolated: now also C14.2, C15.2, C30.2, C32.2, C6.2, C7.2, C9.2, IC2.1 (VOUT)
- net +5V renamed +5V Isolated
- net +5V Isolated: now also IC14.8 (+VS), C10.2, C20.1, C23.1, C24.1, C25.1, C27.1, C50.2, C51.2, C54.2, C56.2, IC3.1 (VOUT)
- net Gate Drive CS renamed Gate Drive ~{CS}
- net Gate Drive ~{CS}: now also IC12.14 (OUTA)
- net Gate Drive LDAC renamed Gate Drive ~{LDAC}
- net Gate Drive ~{LDAC}: now also IC12.11 (OUTD)
- net Sense CS renamed Sense ~{CS}
- net Sense ~{CS}: now also IC9.14 (OUTA)
- net Sense Dout renamed Sense Dout/~{Ready}
- net Sense Dout/~{Ready}: now also IC9.11 (IND)
- new net: L1.2, PS2.6 (+VOUT)
- new net: C4.2, IC4.8 (VIN), PS4.4 (+VOUT)
- new net: L2.2, PS1.5 (+VOUT)
- new net: C2.2, C5.2, IC2.8 (VIN), L2.1
- new net: C3.2, IC3.8 (VIN), PS3.4 (+VOUT)
- new net DGND Isolated: C17.2, C19.2, C20.2, C21.2, C35.1, C36.2, C37.2, C39.1, C40.2, C49.2, C52.2, IC12.15 (GND2_2), IC12.9 (GND2_1), IC13.2 (GND1_1), IC13.7 (EN1), IC13.8 (GND1_2), IC8.17 (DGND), IC9.15 (GND2_2), IC9.9 (GND2_1)
- new net GND Isolated: C1.1, C10.1, C11.1, C12.1, C13.2, C14.1, C15.1, C16.1, C17.1, C18.1, C19.1, C2.1, C22.2, C23.2, C24.2, C25.2, C26.1, C27.2, C28.1, C3.1, C30.1, C32.1, C38.1, C4.1, C41.2, C42.2, C43.2, C44.2, C45.1, C46.1, C47.1, C5.1, C50.1, C51.1, C54.1, C55.1, C56.1, C57.1, C6.1, C7.1, C8.1, C9.1, D1.2 (A), IC1.3 (GND_1), IC1.4 (GND_2), IC1.5 (GND_3), IC1.8 (GND_4), IC10.4 (V-), IC11.3 (GND_1), IC11.4 (GND_2), IC11.5 (GND_3), IC11.8 (GND_4), IC14.5 (-VS), IC15.4 (V-), IC16.2 (GND), IC2.2 (GND_1), IC2.3 (GND_2), IC2.6 (GND_3), IC2.7 (GND_4), IC3.2 (GND_1), IC3.3 (GND_2), IC3.6 (GND_3), IC3.7 (GND_4), IC4.2 (GND_1), IC4.3 (GND_2), IC4.6 (GND_3), IC4.7 (GND_4), IC6.12 (DGND), IC6.3 (AGNDF), IC6.4 (AGNDS), IC7.3 (GND_1), IC7.4 (GND_2), IC7.5 (GND_3), IC7.8 (GND_4), IC8.2 (REF-), IC8.6 (AVSS), PS1.7 (-VOUT), PS2.4 (-VOUT), PS3.3 (-VOUT), PS4.3 (-VOUT), Q1.3 (DS), RV1.2, RV2.2
- no-connect marks 14 -> 48
Other:
- note added: "Data Isolation"
- note added: "Power Conversion + Isolation"
- moved on the sheet: A1, D2, IC10, IC11, IC14, IC15, IC16, IC6, IC7, IC8, Q1, R4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

Commit message: Got the PCB layed out exlucing the grounds
Parts:
- removed C10, C49, C53: 0.1u, symbol Device:C
- removed C3: 0.33u, symbol Device:C
- removed C31: 540p, symbol Device:C
- removed IC13: ISO7741FQDBQRQ1, SOP64P600X175-16N, symbol ISO7741FQDBQRQ1:ISO7741FQDBQRQ1
- removed IC3: L78L05ACD13TR, SOIC127P600X175-8N, symbol L78L05ACD13TR:L78L05ACD13TR
- removed PS3: TBA_1-1219, TBA1, symbol TBA_1-1219:TBA_1-1219
- removed R3: PCS-0R0047D1, symbol Device:R_Shunt_US
- removed RV1: Gate_Drive_Amp_Gain_Adjust 4.7k, symbol Device:R_Potentiometer_Trim
- added C21, C22, C23, C55: 1u, Capacitor_SMD:C_1206_3216Metric, symbol Device:C
- added C27, C28: 0.33u, Capacitor_SMD:C_0805_2012Metric, symbol Device:C
- added C29: 0.1u, Capacitor_SMD:C_0805_2012Metric, symbol Device:C
- added C33: 540p, Capacitor_SMD:C_1210_3225Metric, symbol Device:C
- added C37, C38, C56: 0.1u, Capacitor_SMD:C_0603_1608Metric, symbol Device:C
- added D1: D, S2A:DIOM5336X245N, symbol Device:D
- added H1: RA-T2X-64E, RA-T2X-64E:RAT2X64E, symbol RA-T2X-64E:RA-T2X-64E
- added H2: VM1-038-1AE, VM1-038-1AE:VM1-038-1AE, symbol VM1-038-1AE:VM1-038-1AE
- added IC9: L78L05ACD13TR, L78L05ACD13TR:SOIC127P600X175-8N, symbol L78L05ACD13TR:L78L05ACD13TR
- added J1: Conn_01x03, Connector_PinHeader_2.54mm:PinHeader_1x03_P2.54mm_Vertical, symbol Connector_Generic:Conn_01x03
- added J2: Conn_01x06, Connector_PinHeader_2.54mm:PinHeader_1x06_P2.54mm_Vertical, symbol Connector_Generic:Conn_01x06
- added J3: Fan, 1190363:1190363, symbol 1190363:1190363
- added J4: Power In, 1190363:1190363, symbol 1190363:1190363
- added J5: 1904147, 1904147:1904147, symbol 1904147:1904147
- added J7: UI, 1190363:1190363, symbol 1190363:1190363
- added L3, L4: 47u, 11R473C_47uH:11R473C, symbol Device:L
- added NT1: Isolated Ground Tie, NetTie:NetTie-3_SMD_Pad2.0mm, symbol Device:NetTie_3_Tee
- added NT2: NetTie_2, NetTie:NetTie-2_SMD_Pad2.0mm, symbol Device:NetTie_2
- added PS3: NMA1209SC, NMA1209SC:NMA1209SC, symbol NMA1209SC:NMA1209SC
- added R3: PCS-0R0047D1, PCBLIB_RES-TH_L22.3-W4.5-P7.62-L_2025-03-21:RES-TH_L22.3-W4.5-P7.62-L, symbol SCHLIB_PCS-0R0047D1_2025-03-21:PCS-0R0047D1
- added RV1: A0_Trim, 3386G-1-472LF_Trim_Pot:3386G1503LF, symbol 3386G-1-472LF:3386G-1-472LF
- added RV2: A1_Trim, 3386G-1-472LF_Trim_Pot:3386G1503LF, symbol 3386G-1-472LF:3386G-1-472LF
- added RV3: A2_Trim, 3386G-1-472LF_Trim_Pot:3386G1503LF, symbol 3386G-1-472LF:3386G-1-472LF
- added U1: DI79L05UAB, Package_TO_SOT_SMD:SOT-89-3, symbol DI79L05UAB:DI79L05UAB
- C1: renamed from C6; footprint (none) -> Capacitor_SMD:C_0805_2012Metric
- C10: renamed from C17; footprint (none) -> Capacitor_SMD:C_1206_3216Metric
- C11: renamed from C24; footprint (none) -> Capacitor_SMD:C_0603_1608Metric
- C12: renamed from C25; footprint (none) -> Capacitor_SMD:C_0805_2012Metric
- C13: renamed from C18; footprint (none) -> Capacitor_SMD:C_0603_1608Metric
- C14: renamed from C19; footprint (none) -> Capacitor_SMD:C_0603_1608Metric
- C15: renamed from C20; footprint (none) -> Capacitor_SMD:C_0603_1608Metric
- C16: renamed from C21; footprint (none) -> Capacitor_SMD:C_0603_1608Metric
- C17: renamed from C27; footprint (none) -> Capacitor_SMD:C_0805_2012Metric
- C18: renamed from C22; footprint (none) -> Capacitor_SMD:C_0603_1608Metric
- C19: renamed from C1; footprint (none) -> Capacitor_SMD:C_1206_3216Metric
- C2: renamed from C7; footprint (none) -> Capacitor_SMD:C_0603_1608Metric
- C20: renamed from C2; footprint (none) -> Capacitor_SMD:C_0805_2012Metric
- C24: renamed from C4; footprint (none) -> Capacitor_SMD:C_0805_2012Metric
- C25: renamed from C26; footprint (none) -> Capacitor_SMD:C_0805_2012Metric
- C26: renamed from C5; footprint (none) -> Capacitor_SMD:C_0805_2012Metric
- C3: renamed from C11; footprint (none) -> Capacitor_SMD:C_0603_1608Metric
- C30: renamed from C28; footprint (none) -> Capacitor_SMD:C_0603_1608Metric
- C31: renamed from C38; footprint (none) -> Capacitor_SMD:C_0805_2012Metric
- C32: renamed from C30; footprint (none) -> Capacitor_SMD:C_0805_2012Metric
- C34: renamed from C45; footprint (none) -> Capacitor_SMD:C_1206_3216Metric
- C35: renamed from C8; footprint (none) -> Capacitor_SMD:C_0603_1608Metric
- C36: renamed from C9; footprint (none) -> Capacitor_SMD:C_0603_1608Metric
- C39: renamed from C32; footprint (none) -> Capacitor_SMD:C_0603_1608Metric
- C4: renamed from C12; footprint (none) -> Capacitor_SMD:C_0805_2012Metric
- C40: renamed from C33; footprint (none) -> Capacitor_SMD:C_0603_1608Metric
- C41: renamed from C34; footprint (none) -> Capacitor_SMD:C_0603_1608Metric
- C42: renamed from C35; footprint (none) -> Capacitor_SMD:C_1206_3216Metric
- C43: renamed from C36; footprint (none) -> Capacitor_SMD:C_1206_3216Metric
- C44: renamed from C39; footprint (none) -> Capacitor_SMD:C_0603_1608Metric
- C45: renamed from C40; footprint (none) -> Capacitor_SMD:C_0603_1608Metric
- C46: renamed from C41; footprint (none) -> Capacitor_SMD:C_0603_1608Metric
- C47: renamed from C42; footprint (none) -> Capacitor_SMD:C_0603_1608Metric
- C48: renamed from C43; footprint (none) -> Capacitor_SMD:C_0603_1608Metric
- C49: renamed from C44; footprint (none) -> Capacitor_SMD:C_0603_1608Metric
- C5: renamed from C13; footprint (none) -> Capacitor_SMD:C_0805_2012Metric
- C50: renamed from C46; footprint (none) -> Capacitor_SMD:C_0805_2012Metric
- C51: renamed from C47; footprint (none) -> Capacitor_SMD:C_0603_1608Metric
- C52: renamed from C48; footprint (none) -> Capacitor_SMD:C_0603_1608Metric
- C53: renamed from C29; footprint (none) -> Capacitor_SMD:C_0603_1608Metric
- C54: renamed from C50; footprint (none) -> Capacitor_SMD:C_0805_2012Metric
- C57: renamed from C51; footprint (none) -> Capacitor_SMD:C_0603_1608Metric
- C58: renamed from C52; footprint (none) -> Capacitor_SMD:C_0603_1608Metric
- C59: renamed from C37; footprint (none) -> Capacitor_SMD:C_0603_1608Metric
- C6: renamed from C14; footprint (none) -> Capacitor_SMD:C_0805_2012Metric
- C60: renamed from C54; footprint (none) -> Capacitor_SMD:C_0805_2012Metric
- C61: renamed from C55; footprint (none) -> Capacitor_SMD:C_0603_1608Metric
- C62: renamed from C56; footprint (none) -> Capacitor_SMD:C_0603_1608Metric
- C63: renamed from C57; footprint (none) -> Capacitor_SMD:C_1206_3216Metric
- C7: renamed from C15; footprint (none) -> Capacitor_SMD:C_0603_1608Metric
- C8: renamed from C23; footprint (none) -> Capacitor_SMD:C_0603_1608Metric
- C9: renamed from C16; footprint (none) -> Capacitor_SMD:C_1206_3216Metric
- D2: renamed from D1; footprint HPZRC21QX -> HPZR-C21-QX:HPZRC21QX
- D3: renamed from D2; footprint IXBOD108 -> IXBOD1-08:IXBOD108
- IC1: footprint SOP65P490X110-8N -> REF7050QDGKR:SOP65P490X110-8N
- IC10: renamed from IC11; footprint SOP65P490X110-8N -> REF7050QDGKR:SOP65P490X110-8N
- IC11: renamed from IC12; footprint SOP64P600X175-16N -> ISO7740FQDBQRQ1:SOP64P600X175-16N
- IC12: renamed from IC9; footprint SOP64P600X175-16N -> ISO7741FQDBQRQ1:SOP64P600X175-16N
- IC13: renamed from IC14; footprint SOIC127P600X175-8N -> INA296A3IDDFR:SOT65P280X110-8N
- IC14: renamed from IC15; footprint SOP65P490X110-8N -> OPA210IDGKR:SOP65P490X110-8N
- IC15: renamed from IC16; footprint SOT65P280X110-8N -> INA296A3IDDFR:SOT65P280X110-8N
- IC2: renamed from IC6; footprint SOIC127P600X175-14N -> MAX5719GSD+:SOIC127P600X175-14N
- IC3: renamed from IC7; footprint SOP65P490X110-8N -> REF7050QDGKR:SOP65P490X110-8N
- IC4: renamed from IC8; footprint SOP65P640X120-24N -> AD7175-2BRUZ:SOP65P640X120-24N
- IC5: renamed from IC10; footprint SOP65P490X110-8N -> OPA210IDGKR:SOP65P490X110-8N
- IC6: renamed from IC4; footprint SOIC127P600X175-8N -> L78L33ACD13TR:SOIC127P600X175-8N
- IC7: renamed from IC5; footprint SOIC127P600X175-8N -> L78L33ACD13TR:SOIC127P600X175-8N
- IC8: renamed from IC2; footprint SOIC127P600X175-8N -> L78L06ACD13TR:SOIC127P600X175-8N
- L1: footprint (none) -> 11R473C_47uH:11R473C
- L2: footprint (none) -> 11R683C_68uH:11R683C
- PS1: footprint NKE0503DC -> NKE1212DC:NKE0503DC
- PS2: footprint NMG0524SC -> NMG1212SC:NMG0524SC
- PS4: footprint TBA1 -> TBA_1-1219:TBA1
- R1, R2: footprint (none) -> Resistor_SMD:R_1206_3216Metric
- R4: footprint (none) -> Resistor_SMD:R_2512_6332Metric
- R5: footprint (none) -> Resistor_SMD:R_0805_2012Metric
- RV4: renamed from RV2; footprint (none) -> 3386G-1-472LF_Trim_Pot:3386G1503LF; symbol Device:R_Potentiometer_Trim -> 3386G-1-472LF:3386G-1-472LF; Height (none) -> 4.83; Manufacturer_Name (none) -> Bourns; Manufacturer_Part_Number (none) -> 3386G-1-472LF; Mouser Part Number (none) -> 652-3386G-1-472LF; Mouser Price/Stock (none) -> https://www.mouser.co.uk/ProductDetail/Bourns/3386G-1-472LF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
Connections:
- net +12V: now also D1.2 (A), J3.1, J4.1, J7.1, PS3.1 (+VIN); no longer A1.30 (VIN)
- net +3.3V: now also RV1.1 (CCW), RV2.1 (CCW), RV3.1 (CCW)
- net +5V Isolated: now also C37.2, IC9.1 (VOUT)
- net Current Sense +: now also R3.2 (U)
- net Current Sense -: now also R3.3 (U)
- net Current Sense Amp Out: now also IC5.2 (-IN)
- net DGND Isolated: now also C12.2, IC2.12 (DGND), NT1.1; no longer C15.2, C16.2
- net GND: now also J3.3, J4.3, J7.3, PS3.2 (-VIN), RV1.3 (CW), RV2.3 (CW), RV3.3 (CW)
- net GND Isolated: now also C21.1, C22.1, C27.1, C28.1, C37.1, C38.1, IC9.2 (GND_1), IC9.3 (GND_2), IC9.6 (GND_3), IC9.7 (GND_4), NT1.3, PS3.5 (OV), U1.1 (GND); no longer C1.1, C10.1, C11.2, C12.2, C13.1, C14.1, C17.2, C18.2, C2.1, C25.1, C3.1, C30.1, C31.1, C32.1, C34.1, C39.1, C4.1, C46.2, C47.2, C48.2, C49.2, C5.2, C50.1, C51.1, C54.1, C57.1, C6.1, C60.1, C61.1, C62.1, C63.1, C7.1, C8.2, C9.1, D2.2 (A), IC1.3 (GND_1), IC1.4 (GND_2), IC1.5 (GND_3), IC1.8 (GND_4), IC10.3 (GND_1), IC10.4 (GND_2), IC10.5 (GND_3), IC10.8 (GND_4), IC13.5 (-VS), IC14.4 (V-), IC15.2 (GND), IC2.12 (DGND), IC2.3 (AGNDF), IC2.4 (AGNDS), IC3.3 (GND_1), IC3.4 (GND_2), IC3.5 (GND_3), IC3.8 (GND_4), IC4.2 (REF-), IC4.6 (AVSS), IC5.4 (V-), Q1.3 (DS), RV4.2
- net Gate Drive +: now also C33.2; no longer IC5.6 (OUT)
- net Gate Drive ~{CS} uC: now also A1.9 (D6), IC11.6 (IND); no longer A1.12 (D9), IC11.3 (INA)
- net Gate Drive ~{LDAC} uC: now also A1.12 (D9), IC11.3 (INA); no longer A1.11 (D8), IC11.6 (IND)
- net Sense Amp Ref: now also C41.2, C48.1, IC4.22 (AIN1); no longer C41.1, C49.1, IC4.21 (AIN0)
- net Sense ~{CS} uC: now also A1.8 (D5); no longer A1.13 (D10/CS)
- net Voltage Sense -: now also J5.1, R3.4 (I)
- net Voltage Sense Amp Out: now also C41.1, C49.1, IC4.21 (AIN0); no longer C41.2, C48.1, IC4.22 (AIN1)
- net in+: now also J5.2
- net at A1.19 (A0): now also RV1.2 (WIPER)
- net at A1.20 (A1): now also RV2.2 (WIPER)
- net at A1.21 (A2): now also RV3.2 (WIPER)
- net at A1.22 (A3): now also J2.5 (Pin_5)
- net at A1.23 (SDA/A4): now also J2.4 (Pin_4)
- net at A1.24 (SCL/A5): now also J2.3 (Pin_3)
- net at A1.25 (A6): now also J2.2 (Pin_2)
- net at A1.26 (A7): now also J2.1 (Pin_1)
- net Sense CIPO uC: now reaches A1.5 (D2)
- net Sense CIPO uC: now also IC12.6 (OUTD)
- net Sense COPI uC: now reaches A1.6 (D3)
- net Sense COPI uC: now also IC12.5 (INC)
- net Sense SCLK uC: now reaches A1.7 (D4)
- net Sense SCLK uC: now also IC12.4 (INB)
- net at R1.1: now also IC5.6 (OUT); no longer IC5.2 (-IN)
- net at Q1.2 (S): now also R3.1 (I)
- net at IC14.3 (+IN), R2.1: now also RV4.1 (CCW); no longer RV4.3
- net AGND Isolated: now reaches IC4.1 (AIN4)
- net AGND Isolated: now also C1.1, C10.1, C11.2, C13.1, C14.1, C15.2, C16.2, C17.2, C18.2, C2.1, C25.1, C3.1, C30.1, C31.1, C32.1, C34.1, C39.1, C4.1, C46.2, C47.2, C48.2, C49.2, C5.2, C50.1, C51.1, C54.1, C57.1, C6.1, C60.1, C61.1, C62.1, C63.1, C7.1, C8.2, C9.1, IC1.3 (GND_1), IC1.4 (GND_2), IC1.5 (GND_3), IC1.8 (GND_4), IC10.3 (GND_1), IC10.4 (GND_2), IC10.5 (GND_3), IC10.8 (GND_4), IC13.5 (-VS), IC15.2 (GND), IC2.3 (AGNDF), IC2.4 (AGNDS), IC3.3 (GND_1), IC3.4 (GND_2), IC3.5 (GND_3), IC3.8 (GND_4), IC4.2 (REF-), IC4.6 (AVSS), RV4.2 (WIPER), RV4.3 (CW), C23.1, C29.1, C55.1, C56.1, NT1.2, NT2.1
- net CIPO uC: no longer names the net of A1.15 (D12/CIPO)
- net CIPO uC: now also J1.3 (Pin_3); no longer IC12.6 (OUTD)
- removed net COPI uC: A1.14 (D11/COPI), IC11.5 (INC), IC12.5 (INC)
- removed net SCLK uC: A1.16 (D13/SCK), IC11.4 (INB), IC12.4 (INB)
- net Sense GPIO0: no longer names the net of IC4.20 (GPIO1)
- net Sense GPIO1: no longer names the net of IC4.19 (GPIO0)
- net Sense ~{Error}: no longer names the net of IC4.15 (~{SYNC}/~{ERROR})
- net Sense ~{Error} uC renamed Gate Drive SCLK uC
- net Gate Drive SCLK uC: now also IC11.5 (INC)
- new net: A1.30 (VIN), D1.1 (K)
- new net: C21.2, C27.2, IC9.8 (VIN), L3.1
- new net: L3.2, PS3.6 (+VOUT)
- new net: C22.2, C28.2, L4.1, U1.2 (VIN)
- new net: A1.13 (D10/CS), J1.1 (Pin_1)
- new net: A1.14 (D11/COPI), J1.2 (Pin_2)
- new net: A1.16 (D13/SCK), J2.6 (Pin_6)
- new net: L4.2, PS3.4 (-VOUT)
- new net -5V Isolated: C23.2, C29.2, C38.2, C55.2, C56.2, IC14.4 (V-), IC5.4 (V-), U1.3 (VOUT)
- new net Gate Drive -: C33.1, D2.2 (A), NT2.2, Q1.3 (DS)
- new net Gate Drive COPI uC: A1.11 (D8), IC11.4 (INB)
- no-connect marks 48 -> 43
Other:
- moved on the sheet: A1, C1, C11, C12, C17, C19, C2, C20, C24, C26, C3, C31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

Commit message: Finished laying out all the traces and adding the temperature sensing circuitry
Parts:
- removed J1: Conn_01x03, Connector_PinHeader_2.54mm:PinHeader_1x03_P2.54mm_Vertical, symbol Connector_Generic:Conn_01x03
- removed NT1: Isolated Ground Tie, NetTie:NetTie-3_SMD_Pad2.0mm, symbol Device:NetTie_3_Tee
- added C64, C65, C66, C67, C68: 0.1u, Capacitor_SMD:C_0603_1608Metric, symbol Device:C
- added IC16: MAX31850K, Adafruit:MAX31850K, symbol Adafruit:MAX31850K
- added IC17, IC18: ISO7741FQDBQRQ1, ISO7741FQDBQRQ1:SOP64P600X175-16N, symbol ISO7741FQDBQRQ1:ISO7741FQDBQRQ1
- added NT3: NetTie_2, NetTie:NetTie-2_SMD_Pad2.0mm, symbol Device:NetTie_2
- added R6: 4.7k, Resistor_SMD:R_1206_3216Metric, symbol Device:R
Connections:
- net AGND Isolated is gone; now on net GND Isolated: C1.1, C10.1, C11.2, C13.1, C14.1, C15.2, C16.2, C17.2, C18.2, C2.1, C23.1, C25.1, C29.1, C3.1, C30.1, C31.1, C32.1, C34.1, C39.1, C4.1, C46.2, C47.2, C48.2, C49.2, C5.2, C50.1, C51.1, C54.1, C55.1, C56.1, C57.1, C6.1, C60.1, C61.1, C62.1, C63.1, C7.1, C8.2, C9.1, IC1.3 (GND_1), IC1.4 (GND_2), IC1.5 (GND_3), IC1.8 (GND_4), IC10.3 (GND_1), IC10.4 (GND_2), IC10.5 (GND_3), IC10.8 (GND_4), IC13.5 (-VS), IC15.2 (GND), IC2.3 (AGNDF), IC2.4 (AGNDS), IC3.3 (GND_1), IC3.4 (GND_2), IC3.5 (GND_3), IC3.8 (GND_4), IC4.1 (AIN4), IC4.2 (REF-), IC4.6 (AVSS), NT2.1, RV4.2 (WIPER), RV4.3 (CW)
- net +3.3V: now also C64.2, C65.1, C66.1, IC17.1 (VCC1), IC18.1 (VCC1)
- net +3.3V Isolated: now also C67.1, C68.1, IC16.5 (3V3), IC17.10 (EN2), IC17.16 (VCC2), IC18.16 (VCC2), R6.1; no longer C61.2, C63.2, IC14.7 (V+)
- net +6V Isolated: now also C61.2, C63.2, IC14.7 (V+)
- net DGND Isolated: now also C67.2, C68.2, IC16.3 (GND), IC17.15 (GND2_2), IC17.9 (GND2_1), IC18.15 (GND2_2), IC18.9 (GND2_1), NT3.2
- net GND: now also C64.1, C65.2, C66.2, IC17.2 (GND1_1), IC17.8 (GND1_2), IC18.2 (GND1_1), IC18.7 (EN1), IC18.8 (GND1_2)
- net GND Isolated: now also NT3.1
- net Temp Write EN uC: now reaches A1.13 (D10/CS)
- net Temp Write EN uC: now also IC17.3 (INA)
- net Temp Sensor uC: now reaches A1.14 (D11/COPI)
- net Temp Sensor uC: now also IC17.6 (OUTD), IC18.3 (INA)
- net Temp Read EN uC: now reaches A1.15 (D12/CIPO)
- net Temp Read EN uC: now also IC17.7 (EN1)
- new net Temp Sensor: IC16.10 (DATA), IC17.11 (IND), IC18.14 (OUTA), R6.2
- new net Temp Write EN: IC17.14 (OUTA), IC18.10 (EN2)
- no-connect marks 43 -> 60
Other:
- moved on the sheet: C52, C53, C58, C59, IC11, IC12
