File: DC Load.kicad_pcb (KiCad board)
At the start: 2 copper layers, 225 x 180 mm, 160 parts, among them IC1 REF7050QDGKR, IC10 REF7050QDGKR, IC11 ISO7740FQDBQRQ1, IC12 ISO7741FQDBQRQ1, IC13 INA826AID, IC14 OPA210IDGKR, IC15 INA296A3IDDFR, IC16 MAX31850K, IC17 ISO7741FQDBQRQ1, IC18 ISO7741FQDBQRQ1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

Commit message: fixed net names for DAC communincation
Connections:
- A1 pad 10: Gate Drive SCLK uC -> Gate Drive COPI uC
- A1 pad 11: Gate Drive COPI uC -> Gate Drive SCLK uC
- A1 pad 12: Gate Drive ~{LDAC} uC -> Gate Drive ~{CS} uC
- A1 pad 9: Gate Drive ~{CS} uC -> Gate Drive ~{LDAC} uC
- IC11 pad 3: Gate Drive ~{LDAC} uC -> Gate Drive ~{CS} uC
- IC11 pad 4: Gate Drive COPI uC -> Gate Drive SCLK uC
- IC11 pad 5: Gate Drive SCLK uC -> Gate Drive COPI uC
- IC11 pad 6: Gate Drive ~{CS} uC -> Gate Drive ~{LDAC} uC
Changed lines of the file:
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@@
 			(size 0.435 1.528)
 			(layers "F.Cu" "F.Paste" "F.Mask")
-			(net 4 "Gate Drive ~{LDAC} uC")
+			(net 5 "Gate Drive ~{CS} uC")
 			(pinfunction "INA")
 			(pintype "passive")
@@
 			(size 0.435 1.528)
 			(layers "F.Cu" "F.Paste" "F.Mask")
-			(net 11 "Gate Drive COPI uC")
+			(net 1 "Gate Drive SCLK uC")
 			(pinfunction "INB")
 			(pintype "passive")
@@
 			(size 0.435 1.528)
 			(layers "F.Cu" "F.Paste" "F.Mask")
-			(net 1 "Gate Drive SCLK uC")
+			(net 11 "Gate Drive COPI uC")
 			(pinfunction "INC")
 			(pintype "passive")
@@
 			(size 0.435 1.528)
 			(layers "F.Cu" "F.Paste" "F.Mask")
-			(net 5 "Gate Drive ~{CS} uC")
+			(net 4 "Gate Drive ~{LDAC} uC")
 			(pinfunction "IND")
 			(pintype "passive")
@@
 			(layers "*.Cu" "*.Mask")
 			(remove_unused_layers no)
-			(net 5 "Gate Drive ~{CS} uC")
+			(net 4 "Gate Drive ~{LDAC} uC")
 			(pinfunction "D6")
 			(pintype "bidirectional")
@@
 			(layers "*.Cu" "*.Mask")
 			(remove_unused_layers no)
-			(net 1 "Gate Drive SCLK uC")
+			(net 11 "Gate Drive COPI uC")
 			(pinfunction "D7")
 			(pintype "bidirectional")
@@
 			(layers "*.Cu" "*.Mask")
 			(remove_unused_layers no)
-			(net 11 "Gate Drive COPI uC")
+			(net 1 "Gate Drive SCLK uC")
 			(pinfunction "D8")
 			(pintype "bidirectional")
@@
 			(layers "*.Cu" "*.Mask")
 			(remove_unused_layers no)
-			(net 4 "Gate Drive ~{LDAC} uC")
+			(net 5 "Gate Drive ~{CS} uC")
 			(pinfunction "D9")
 			(pintype "bidirectional")
@@
 	)
 	(segment
-		(start 85.6 144.94)
-		(end 109.831962 144.94)
+		(start 110.585375 143.085375)
+		(end 109.9 142.4)
 		(width 0.3)
 		(layer "F.Cu")
@@
 	)
 	(segment
-		(start 109.831962 144.94)
-		(end 111.050587 143.721375)
+		(start 112.032625 143.085375)
+		(end 110.585375 143.085375)
 		(width 0.3)
 		(layer "F.Cu")
@@
 	)
 	(segment
-		(start 111.050587 143.721375)
-		(end 112.032625 143.721375)
+		(start 109.9 142.4)
+		(end 85.6 142.4)
 		(width 0.3)
 		(layer "F.Cu")
@@
 	)
 	(segment
-		(start 108.26 139.86)
-		(end 110.137288 141.737288)
+		(start 107.9425 147.48)
+		(end 111.067125 144.355375)
 		(width 0.3)
 		(layer "F.Cu")
@@
 	)
 	(segment
-		(start 110.854087 142.451375)
-		(end 112.032625 142.451375)
+		(start 85.6 147.48)
+		(end 107.9425 147.48)
 		(width 0.3)
 		(layer "F.Cu")
@@
 	)
 	(segment
-		(start 110.137288 141.737288)
-		(end 110.14 141.737288)
+		(start 111.067125 144.355375)
+		(end 112.032625 144.355375)
 		(width 0.3)
 		(layer "F.Cu")
@@
 	)
 	(segment
-		(start 110.14 141.737288)
-		(end 110.854087 142.451375)
+		(start 108.26 139.86)
+		(end 110.137288 141.737288)
 		(width 0.3)
 		(layer "F.Cu")
-		(net 4)
+		(net 5)
 	)
 	(segment
-		(start 85.6 139.86)
-		(end 108.26 139.86)
+		(start 110.854087 142.451375)
+		(end 112.032625 142.451375)
 		(width 0.3)
 		(layer "F.Cu")
-		(net 4)
+		(net 5)
 	)
 	(segment
-		(start 107.9425 147.48)
-		(end 111.067125 144.355375)
+		(start 110.137288 141.737288)
+		(end 110.14 141.737288)
 		(width 0.3)
 		(layer "F.Cu")
@@
 	)
 	(segment
-		(start 85.6 147.48)
-		(end 107.9425 147.48)
+		(start 110.14 141.737288)
+		(end 110.854087 142.451375)
 		(width 0.3)
 		(layer "F.Cu")
@@
 	)
 	(segment
-		(start 111.067125 144.355375)
-		(end 112.032625 144.355375)
+		(start 85.6 139.86)
+		(end 108.26 139.86)
 		(width 0.3)
 		(layer "F.Cu")
@@
 	)
 	(segment
-		(start 110.585375 143.085375)
-		(end 109.9 142.4)
+		(start 85.6 144.94)
+		(end 109.831962 144.94)
 		(width 0.3)
 		(layer "F.Cu")
@@
 	)
 	(segment
-		(start 112.032625 143.085375)
-		(end 110.585375 143.085375)
+		(start 109.831962 144.94)
+		(end 111.050587 143.721375)
 		(width 0.3)
 		(layer "F.Cu")
@@
 	)
 	(segment
-		(start 109.9 142.4)
-		(end 85.6 142.4)
+		(start 111.050587 143.721375)
+		(end 112.032625 143.721375)
 		(width 0.3)
 		(layer "F.Cu")
